Commit message: snapshot

File: pan_tilt_desc/urdf/pt_1.0.urdf (robot description, URDF)
Before this commit: robot pan_tilt, 4 links, 3 joints
Links:
- link base_assembly: geometry visual mesh filename=package://pan_tilt_desc/stl/pt_1.0/pt_base_assembly.stl scale=0.001 0.001 0.001
- link pan_assembly: geometry visual mesh filename=package://pan_tilt_desc/stl/pt_1.0/pt_pan_assembly.stl scale=0.001 0.001 0.001
- link tilt_assembly: geometry visual mesh filename=package://pan_tilt_desc/stl/pt_1.0/pt_tilt_assembly.stl scale=0.001 0.001 0.001
Joints:
- joint tilt: origin xyz=0 0 67.0 rpy=0 0 0 -> xyz=0 0 0.067 rpy=0 0 0
